File: phrog-mainboard/_autosave-phrog-mainboard.kicad_sch (KiCad schematic)
At the start: 52 parts, among them J1 Battery, Q1 2N7000, Q2 2N7000, SW1 SW_Push, SW3 SW_SPDT, U1 NRF52840 Pro Micro, U2 LM358, U3 NAU7802KGI, U4 MCP34063

Commit message: start routing PCB
Parts:
- U4: value MCP34063 -> MC34063
Other:
- note added: "Update resistor values for the LEDs!"
Changed lines of the file:
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@@
 		)
 	)
+	(text "Update resistor values for the LEDs!\n"
+		(exclude_from_sim no)
+		(at 251.46 106.426 0)
+		(effects
+			(font
+				(size 1.27 1.27)
+			)
+		)
+	)
 	(junction
 		(at 166.37 20.32)
@@
 			)
 		)
-		(property "Value" "MCP34063"
+		(property "Value" "MC34063"
 			(at 186.436 24.13 0)
 			(show_name no)
