File: phrog-mainboard/phrog-mainboard.kicad_pcb (KiCad board)
At the start: 2 copper layers, 33 parts, among them J1 Battery, Q1 2N7000, Q2 2N7000, SW1 SW_Push, SW3 SW_SPDT, U1 NRF52840 Pro Micro, U2 LM358, U3 NAU7802KGI, U4 MCP34063

Commit message: finish first draft of enclosure
Parts:
- removed L1: 510uH, Inductor_THT:L_Axial_L11.0mm_D4.5mm_P15.24mm_Horizontal_Fastron_MECC
- removed Q1, Q2: 2N7000, Package_TO_SOT_THT:TO-92_Inline
- removed R3: 2.7R, Resistor_THT:R_Axial_DIN0207_L6.3mm_D2.5mm_P10.16mm_Horizontal
- removed R4: 180R, Resistor_THT:R_Axial_DIN0207_L6.3mm_D2.5mm_P10.16mm_Horizontal
- removed R5: 1k, Resistor_THT:R_Axial_DIN0207_L6.3mm_D2.5mm_P10.16mm_Horizontal
- removed R7: 3k, Resistor_THT:R_Axial_DIN0207_L6.3mm_D2.5mm_P10.16mm_Horizontal
- added D4: 1N5817, Diode_THT:D_DO-41_SOD81_P10.16mm_Horizontal, F.Cu at (89.0, 46.5)
- added G***: LOGO, LOGO, F.Cu at (130.1, 69.5)
- added G***: LOGO, LOGO, B.Cu at (87.0, 77.0)
- added Q3: 2N3904, Package_TO_SOT_THT:TO-92_Inline, F.Cu at (142.0, 50.0)
- added Q4: 2N3904, Package_TO_SOT_THT:TO-92_Inline, F.Cu at (148.3, 77.3)
- added R10: 10k, Resistor_THT:R_Axial_DIN0207_L6.3mm_D2.5mm_P10.16mm_Horizontal, F.Cu at (148.0, 42.0)
- added R11: 5.6k, Resistor_THT:R_Axial_DIN0207_L6.3mm_D2.5mm_P10.16mm_Horizontal, F.Cu at (151.5, 51.9)
- added R12: 10k, Resistor_THT:R_Axial_DIN0207_L6.3mm_D2.5mm_P10.16mm_Horizontal, F.Cu at (141.8, 85.8)
- added R13: 5.6k, Resistor_THT:R_Axial_DIN0207_L6.3mm_D2.5mm_P10.16mm_Horizontal, F.Cu at (144.8, 75.7)
- added REF**: MountingHole_2.2mm_M2_DIN965_Pad, MountingHole:MountingHole_2.2mm_M2_DIN965_Pad, F.Cu at (151.0, 86.5)
- added REF**: MountingHole_2.2mm_M2_DIN965_Pad, MountingHole:MountingHole_2.2mm_M2_DIN965_Pad, F.Cu at (64.8, 87.5)
- added REF**: MountingHole_2.2mm_M2_DIN965_Pad, MountingHole:MountingHole_2.2mm_M2_DIN965_Pad, F.Cu at (119.0, 42.0)
- added REF**: MountingHole_2.2mm_M2_DIN965_Pad, MountingHole:MountingHole_2.2mm_M2_DIN965_Pad, F.Cu at (65.0, 42.0)
- added REF**: MountingHole_2.2mm_M2_DIN965_Pad, MountingHole:MountingHole_2.2mm_M2_DIN965_Pad, F.Cu at (143.5, 42.0)
- added REF**: MountingHole_2.2mm_M2_DIN965_Pad, MountingHole:MountingHole_2.2mm_M2_DIN965_Pad, F.Cu at (132.5, 83.5)
- C4: value 100uF -> 10uF; footprint Capacitor_THT:CP_Radial_D8.0mm_P5.00mm -> Capacitor_THT:C_Disc_D4.3mm_W1.9mm_P5.00mm
- C5: value 510pF -> 10uF
- C6: value 100uF -> 100nF; footprint Capacitor_THT:CP_Radial_D8.0mm_P5.00mm -> Capacitor_THT:C_Disc_D4.3mm_W1.9mm_P5.00mm
- D1: value 1N5818 -> 1N5817
- D2, D3, PD_Blue1, PD_Green1: moved to B.Cu
- R8, R9: value 1k -> 27R
- SW1: value SW_Push -> RESET
- U4: value MCP34063 -> 7660S
- moved U4 30.8 mm to (75.5, 53.0)
- moved R9 28.7 mm to (151.3, 65.3), turned to 180 degrees
- moved U3 26.7 mm to (102.0, 64.1)
- moved C1 26.2 mm to (105.1, 52.1)
- moved C2 26.2 mm to (105.1, 67.6)
- moved C3 26.2 mm to (104.9, 63.7)
- moved RV1 26.2 mm to (114.4, 64.5)
- moved U2 25.7 mm to (107.9, 60.3)
- moved R8 25.3 mm to (151.3, 61.6), turned to 180 degrees
- moved D1 24.7 mm to (89.0, 53.0), turned to 180 degrees
- moved C5 23.0 mm to (88.0, 43.0), turned to 180 degrees
- moved RV2 22.8 mm to (118.0, 48.2)
- moved PD_Green1 22.5 mm to (123.0, 56.8), turned to 90 degrees
- moved PD_Blue1 22.4 mm to (122.6, 71.0), turned to 90 degrees
- moved D2 21.9 mm to (151.4, 57.8), turned to 90 degrees
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Connections:
- C4 pad 1: +BATT -> Net-(D1-K)
- C4 pad 2: GND -> Net-(U4-CAP+)
- C5 pad 1: Net-(U4-TC) -> +5V
- D1 pad 1: +5V -> Net-(D1-K)
- D1 pad 2: Net-(D1-A) -> +BATT
- R8 pad 1: Net-(D2-K) -> Net-(Q3-E)
- R8 pad 2: Net-(Q1-D) -> GND
- R9 pad 1: Net-(D3-K) -> Net-(Q4-E)
- R9 pad 2: Net-(Q2-D) -> GND
- U1 pad 18: /THERM_SIG -> unconnected-(U1-115-Pad18)
- U4 pad 1: Net-(D1-A) -> +BATT
- U4 pad 2: GND -> Net-(U4-CAP+)
- U4 pad 3: Net-(U4-TC) -> GND
- U4 pad 4: GND -> unconnected-(U4-CAP--Pad4)
- U4 pad 5: Net-(U4-CII) -> GND
- U4 pad 6: +BATT -> unconnected-(U4-LV-Pad6)
- U4 pad 7: Net-(U4-IPK) -> unconnected-(U4-OSC-Pad7)
- U4 pad 8: Net-(U4-DRC) -> +BATT
Routing:
- net +5V: track 10.4 -> 107.0 mm
- net /GREEN_DRIVE: track 0.00 -> 94.9 mm, vias 0 -> 4
- net /THERM_SIG: track 0.00 -> 61.9 mm
- net /BLUE_DRIVE: track 0.00 -> 61.5 mm, vias 0 -> 2
- net +3.3V: track 0.00 -> 46.4 mm
- net /SCL: track 0.00 -> 45.4 mm, vias 0 -> 2
- net /DRDY: track 0.00 -> 44.7 mm, vias 0 -> 2
- net /THERM_DRIVE: track 0.00 -> 40.8 mm
- net /SDA: track 0.00 -> 32.3 mm, vias 0 -> 2
- net Net-(U1-RST): track 0.00 -> 20.1 mm
- net Net-(Q3-E): track 0.00 -> 15.4 mm
- net Net-(U4-IPK): track 14.0 -> 0.00 mm
- net Net-(D1-K): track 0.00 -> 13.4 mm
- net Net-(Q4-E): track 0.00 -> 13.3 mm
- net +BATT: track 20.5 -> 32.8 mm
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- added copper zone on B.Cu, net GND
- added copper zone on F.Cu, net GND
Other:
- board outline added: 92.4 x 51 mm
- board text added: "10k"
- board text added: "OFF"
- board text added: "ON"
- board text added: "pHrog Main Board V1.0.0 - {dblquote}BullFrog{dblquote} Jonathan Pfeifer pHalkon Industries 2026-08-30"
